File: sd card copier.sch (EAGLE design)
At the start: 119 parts, among them J2 2x3p-2.54, K1 TS-1188E, K2 TS-1188E, K3 TS-1188E, U1 CJT1117-3.3-SOT223, U4 310090051_24LC32AT-I/OT, Y1 7M-25

Commit message: Submitted for construction at SEEED
Time for bed.
Parts:
- removed C27, C34: (no value), rcl:C-EUC0402
- removed Y1: 7M-25, amino:7M-25
- added C11, C13, C14, C15, C16, C17, C18, C19: 100nf, Seeed-Capacitor:CERAMIC-100NF-50V-10%-X7R(0603)
- added C9: 4.7uf, Seeed-Capacitor:CERAMIC-4.7UF-10V-10%-X5R(0603)
- added D19: YELLOW-0603, Seeed-LED:SMD-LED-CLEAR-YELLOW(0603)
- added DEBUG_TEST, INT_CLK_TEST, TP1, TP2, TP3, TP4, TP5, TP6, TP7: TEST-POINTTP_15TH_THRU, SparkFun-Connectors:TEST-POINTTP_15TH_THRU
- added FD1, FD2, FD3, FD4, FD5, FD6: FIDUCIAL1X2, SparkFun-Aesthetics:FIDUCIAL1X2
- added J3: 2x3p-2.54, Seeed-Connector:DIP-BLACK-MALE-HEADER(2X3P-2.54）-2.54
- added J4, J5: 8p-2.54, Seeed-Connector:DIP-LONG-BLACK-FEMALE-HEADER-VERT(8P-2.54)
- added J7: (no value), Seeed-Connector:DIP-BLACK-JUMPER
- added R22: 3K, Seeed-Resistor:SMD-RES-3K-1%-1/10W(0603)
- added R67, R68, R69, R70, R71, R72, R73, R74, R75, R76, R77, R78, R79, R80, R81, R82, R83, R84, R85, R86, R87: 39R 1/10W, Seeed-Resistor:SMD-RES-39R-5%-1/10W(0603)
- added Y2: 8MHZ, Seeed-Crystal Oscillator:SMD-RESONATOR-8MHZ-33PF-0.1%(3P-3.2X1.3MM)
- C2: value (none) -> 100nf; device rcl:C-EUC0402 -> Seeed-Capacitor:CERAMIC-100NF-50V-10%-X7R(0603)
- C40: device Seeed-Capacitor:CERAMIC-10UF-6.3V-20%-X5R(0402) -> Seeed-Capacitor:CERAMIC-10UF-10V-10%-X5R(0603)
- C6, C7, C8: device Seeed-Capacitor:CERAMIC-4.7UF-6.3V-20%-X5R(0402) -> Seeed-Capacitor:CERAMIC-4.7UF-10V-10%-X5R(0603)
- R14, R15, R20, R21, R23, R28, R29, R30, R44, R45, R46, R51, R52, R53, R6: value 51K -> DNP
- R36, R37: device rcl:R-EU_R0402 -> Seeed-Resistor:SMD-RES-22R-5%-1/10W(0603)
Connections:
- removed net N$18: PI_GPIO.26
- removed net N$8: U$1.VDDA
- removed net SPI_MOSI: J2.3
- new net N$100: DEBUG_TEST.1, U$1.PA14
- new net N$56: D19.+, R22.1
- new net N$57: R67.2, SD2.DI
- new net N$58: R68.2, SD2.SCLK
- new net N$59: R69.2, SD2.DO
- new net N$60: R70.2, SD3.DI
- new net N$61: R71.2, SD3.SCLK
- new net N$62: R72.2, SD3.DO
- new net N$63: R73.2, SD4.DI
- new net N$64: R74.2, SD4.SCLK
- new net N$65: R75.2, SD4.DO
- new net N$66: R76.2, SD5.DI
- new net N$67: R77.2, SD5.SCLK
- new net N$68: R78.2, SD5.DO
- new net N$69: R79.2, SD6.DI
- new net N$70: R80.2, SD6.SCLK
- new net N$71: R81.2, SD6.DO
- new net N$72: R82.2, SD7.DI
- new net N$73: R83.2, SD7.SCLK
- new net N$74: R84.2, SD7.DO
- new net N$75: R85.2, SD8.DI
- new net N$76: R86.2, SD8.SCLK
- new net N$77: R87.2, SD8.DO
- new net N$99: INT_CLK_TEST.1, U$1.PA8
- new net SPI3_!SS: J4.1, U$1.PA15
- new net SPI3_CLK: J4.3, U$1.PB3
- new net SPI3_MISO: J3.2, U$1.PB4
- new net SPI3_MISOPIN: J3.1, J4.5
- new net SPI3_MOSI: J3.6, U$1.PB5
- new net SPI3_MOSIPIN: J3.5, J4.6
- new net STACK1: J5.3, PI_GPIO.12, U$1.PC0
- new net STACK2: J5.4, PI_GPIO.26, U$1.PC13
- new net STACK3: J5.5, PI_GPIO.38, U$1.PC14
- new net STACK4: J5.6, PI_GPIO.40, U$1.PC15
- new net STATUSLED: R22.2, U$1.PA13
- net !RESET: now also C2.2, J7.1, TP2.1; no longer C2.1
- net +3V3: now also C11.1, C13.1, C14.1, C15.1, C16.1, C17.1, C18.1, C19.1, C9.2, J4.7, J4.8, J5.2, J5.7, TP3.1, U$1.VDDA
- net +5V: now also TP5.1
- net BOOT: now also TP1.1
- net GND: now also C11.2, C13.2, C14.2, C15.2, C16.2, C17.2, C18.2, C19.2, C2.1, C9.1, D19.-, J3.3, J3.4, J4.2, J4.4, J5.1, J5.8, J7.2, TP4.1, Y2.2; no longer C2.2, C27.1, C34.1, Y1.GND@1, Y1.GND@2
- net N$19: now also Y2.1; no longer C27.2, Y1.X1
- net N$4: now also USB1.GND@2, USB1.GND@3
- net N$7: now also Y2.3; no longer C34.2, Y1.X2
- net SD2!SS: now also PI_GPIO.3
- net SD3!SS: now also PI_GPIO.5
- net SD4!SS: now also PI_GPIO.29
- net SD4LED: now also U$1.PB6; no longer U$1.PB3
- net SD5!SS: now also PI_GPIO.31
- net SD5LED: now also U$1.PB7; no longer U$1.PB4
- net SD6!SS: now also PI_GPIO.33
- net SD6LED: now also U$1.PB8; no longer U$1.PB5
- net SD7!SS: now also PI_GPIO.35
- net SD7LED: now also U$1.PB9; no longer U$1.PB6
- net SD8!SS: now also PI_GPIO.36
- net SD8LED: now also U$1.PB13; no longer U$1.PB7
- net SPI1_CLK: now also R68.1, R71.1, R74.1, R77.1; no longer SD2.SCLK, SD3.SCLK, SD4.SCLK, SD5.SCLK
- net SPI1_MISO: now also R69.1, R72.1, R75.1, R78.1; no longer SD2.DO, SD3.DO, SD4.DO, SD5.DO
- net SPI1_MOSI: now also J2.3, R67.1, R70.1, R73.1, R76.1; no longer SD2.DI, SD3.DI, SD4.DI, SD5.DI
- net SPI2_!SS: now also TP7.1
- net SPI2_CLK: now also R80.1, R83.1, R86.1; no longer SD6.SCLK, SD7.SCLK, SD8.SCLK
- net SPI2_MISO: now also R81.1, R84.1, R87.1; no longer SD6.DO, SD7.DO, SD8.DO
- net SPI2_MOSI: now also R79.1, R82.1, R85.1; no longer SD6.DI, SD7.DI, SD8.DI
- net VBUS: now also D2.+, TP6.1
Other:
- note added: "MOSI/MISO INVERSION JUMPER FOR SLAVE CARDS"
- note added: "PCB STACKING HEADERS"
- note added: "RESET HOLD JUMPER IF NOT USING STM32"
- note added: "Released under the CERN Open Hardware License Version 1.2"
- note added: "SPI1"
- note added: "SPI2"
- note added: "STM32F401RET6"
- note added: "Thanks to the myStorm guys, I used your STM32 parts as inspiration, and thanks to Oliver for the constructive comments during design!"
- note removed: "STM32F373 or GD32F103"
- note removed: "Thanks to the myStorm guys, I used your STM32 parts as inspiration!"
- note removed: "To do: Check the passives Layout (100x100mm board with everything on the front edge) Consider adding a multiplexer for stacking"
- moved on the sheet: 3V3, C1, C10, C12, C3, C4, C5, C6, C7, C8, D1, D10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
